Commit message: 改了碰撞体，关闭pd和motor stgrenth随机化，关闭倾斜终止

File: legged_gym/resources/robots/adam_pro/adam_pro.urdf (robot description, URDF)
Before this commit: robot adam_pro, 35 links, 34 joints
Links:
- link anklePitchLeft: geometry visual mesh filename=meshes_dae/anklePitchLeft.dae
- link anklePitchRight: geometry visual mesh filename=meshes_dae/anklePitchRight.dae
- link hipRollLeft: geometry visual mesh filename=meshes_dae/hipRollLeft.dae
- link hipRollRight: geometry visual mesh filename=meshes_dae/hipRollRight.dae
- link pelvis: geometry collision cylinder length=0.1 radius=0.1; visual mesh filename=meshes_dae/pelvis.dae
- link shinLeft: geometry collision cylinder length=0.22 radius=0.04; visual mesh filename=meshes_dae/shinLeft.dae
- link shinRight: geometry collision cylinder length=0.22 radius=0.04; visual mesh filename=meshes_dae/shinRight.dae
- link shoulderPitchLeft: geometry visual mesh filename=meshes_dae/shoulderPitchLeft.dae
- link shoulderPitchRight: geometry visual mesh filename=meshes_dae/shoulderPitchRight.dae
- link shoulderRollLeft: geometry collision cylinder length=0.02 radius=0.035; visual mesh filename=meshes_dae/shoulderRollLeft.dae
- link shoulderRollRight: geometry collision cylinder length=0.067 radius=0.0415; visual mesh filename=meshes_dae/shoulderRollRight.dae
- link shoulderYawLeft: geometry collision cylinder length=0.067 radius=0.0415; visual mesh filename=meshes_dae/shoulderYawLeft.dae
- link shoulderYawRight: geometry visual mesh filename=meshes_dae/shoulderYawRight.dae
- link thighLeft: geometry collision cylinder length=0.08 radius=0.06; visual mesh filename=meshes_dae/thighLeft.dae
- link thighRight: geometry collision cylinder length=0.08 radius=0.06; visual mesh filename=meshes_dae/thighRight.dae
- link waistPitch_link: geometry visual mesh filename=meshes_dae/waistPitch_link.dae

Commit message: 碰撞体修正

File: legged_gym/resources/robots/adam_pro/adam_pro.urdf (robot description, URDF)
Before this commit: robot adam_pro, 35 links, 34 joints
Links:
- link wristRollLeft: geometry collision mesh filename=meshes_stl_0.25/wristRollLeft.STL; visual mesh filename=meshes_dae/wristRollLeft.dae
- link wristRollRight: geometry collision mesh filename=meshes_stl_0.25/wristRollRight.STL; visual mesh filename=meshes_dae/wristRollRight.dae

Commit message: 去掉手腕pitch yaw和pitch的碰撞

File: legged_gym/resources/robots/adam_pro/adam_pro.urdf (robot description, URDF)
Before this commit: robot adam_pro, 35 links, 34 joints
Links:
- link wristPitchLeft: geometry visual mesh filename=meshes_dae/wristPitchLeft.dae
- link wristPitchRight: geometry visual mesh filename=meshes_dae/wristPitchRight.dae
- link wristYawLeft: geometry visual mesh filename=meshes_dae/wristYawLeft.dae
- link wristYawRight: geometry visual mesh filename=meshes_dae/wristYawRight.dae

Commit message: 数据集pick put 修正，手部原点修正，config参数修正

File: legged_gym/resources/robots/adam_pro/adam_pro.urdf (robot description, URDF)
Before this commit: robot adam_pro, 35 links, 34 joints
Links:
- added link left_palm_link
- added link right_palm_link
Joints:
- added joint left_palm_joint: type fixed, parent wristRollLeft, child left_palm_link, origin xyz=0.0 -0.0 -0.07 rpy=0 0 0
- added joint right_palm_joint: type fixed, parent wristRollRight, child right_palm_link, origin xyz=0.0 -0.0 -0.07 rpy=0 0 0

Commit message: 箱子变大,相机调整

File: legged_gym/resources/robots/adam_pro/adam_pro.urdf (robot description, URDF)
Before this commit: robot adam_pro, 37 links, 36 joints
Links:
- added link camera_link
Joints:
- added joint camera_joint: type fixed, parent neckPitch_link, child camera_link, origin xyz=0.096 -0.02 0.0407 rpy=0 0 0

Commit message: amp_coef = 0.25  箱子变大 加入小臂碰撞体 取消dual_hand_pos奖励

File: legged_gym/resources/robots/adam_pro/adam_pro.urdf (robot description, URDF)
Before this commit: robot adam_pro, 38 links, 37 joints
Links:
- link wristYawLeft: geometry collision mesh filename=meshes_stl_0.25/wristYawLeft.STL; visual mesh filename=meshes_dae/wristYawLeft.dae
- link wristYawRight: geometry collision mesh filename=meshes_stl_0.25/wristYawRight.STL; visual mesh filename=meshes_dae/wristYawRight.dae

Commit message: 更改wristyaw碰撞体

File: legged_gym/resources/robots/adam_pro/adam_pro.urdf (robot description, URDF)
Before this commit: robot adam_pro, 38 links, 37 joints
Links:
- link wristYawLeft: geometry collision cylinder length=0.1 radius=0.038; visual mesh filename=meshes_dae/wristYawLeft.dae
- link wristYawRight: geometry collision cylinder length=0.1 radius=0.038; visual mesh filename=meshes_dae/wristYawRight.dae
